File: Proyecto_guitarra/guitarra/guitarra.kicad_pcb (KiCad board)
At the start: 2 copper layers, 98.5 x 33.3 mm, 19 parts, among them Q1 2N3904, Q2 2N3904, SW1 SW_SPDT

Commit message: actualizada guitarra
Parts:
- R1, R2: moved to F.Cu
- moved R1 18.0 mm to (103.9, 46.8), turned to -90 degrees
- moved R2 15.6 mm to (106.7, 45.0), turned to 90 degrees
- moved C2 9.81 mm to (98.6, 42.2)
- moved R4 9.50 mm to (98.6, 44.4)
- moved C1 6.67 mm to (95.1, 47.8), turned to 0 degrees
- moved Q1 1.30 mm to (103.2, 42.4), turned to 0 degrees
- moved Q2 1.04 mm to (99.8, 47.6)
- moved REF** 0.65 mm to (127.9, 45.8)
- moved R3 0.31 mm to (95.1, 50.1)
- moved D6 0.10 mm to (135.3, 55.8)
- turned D1 to -90 degrees
- turned D2 to -90 degrees
- turned D3 to -90 degrees
Routing:
- net +3V0: track 48.2 -> 14.3 mm, vias 2 -> 0
- net /sw_on: track 66.5 -> 42.2 mm
- net GND: track 21.2 -> 1.62 mm, vias 1 -> 2
- net /chr_b: track 23.6 -> 5.18 mm
- net /k_a: track 72.1 -> 89.1 mm, vias 6 -> 5
- net /leds_a: track 45.3 -> 60.4 mm, vias 3 -> 4
- net /leds_b: track 63.0 -> 70.5 mm, vias 11 -> 4
- net /chr_a: track 10.9 -> 5.07 mm
- net /k_b: track 86.1 -> 91.1 mm, vias 10 -> 5
- net (no net): track 0.86 -> 0.00 mm

Commit message: drc superado
Parts:
- moved SW1 0.39 mm to (101.2, 68.9)
Connections:
- SW1 pad 3: unconnected-(SW1-C-Pad3) -> (no net)
Routing:
- net /sw_on: track 42.2 -> 38.1 mm
- net GND: vias 2 -> 5

Commit message: release version
Parts:
- added ?: , clipboard:a43f9760-6836-4fde-ab85-758a62f039ea, B.Cu at (97.8, 48.7)
- added G***: LOGO, LOGO, F.Cu at (96.5, 56.0)
- added G***: LOGO, LOGO, F.Cu at (127.3, 46.5)
